File: CabHat_relay.kicad_sch (KiCad schematic)
At the start: 1 part, among them J1 Conn_01x08

Commit message: add sch
Parts:
- added C1: 100n, Library:C_0603_1608Metric, symbol Library:C
- added J2: Barrel_Jack_Switch, symbol Library:Barrel_Jack_Switch
- added JP1, JP2, JP3, JP4: SolderJumper_2_Open, Library:SolderJumper-2_P1.3mm_Open_Pad1.0x1.5mm, symbol Library:SolderJumper_2_Open
- added R1, R2, R3: 10k, Library:R_0603_1608Metric, symbol Library:R
- added U1: PCA9555PW, Library:TSSOP-24_4.4x7.8mm_P0.65mm, symbol Library:PCA9555PW
- J1: lcsc (none) -> x
Connections:
- net +3V3: now also C1.1, JP2.2 (B), JP3.2 (B), JP4.2 (B), U1.24 (VDD)
- net +5V: now also JP1.2 (B)
- net GND: now also C1.2, J2.2, J2.3, R1.2, R2.2, R3.2, U1.12 (VSS)
- net SCL: now reaches J1.6 (Pin_6)
- net SCL: now also U1.22 (SCL)
- net SDA: now reaches J1.7 (Pin_7)
- net SDA: now also U1.23 (SDA)
- new net +VSW: J2.1, JP1.1 (A)
- new net A0: JP2.1 (A), R1.1, U1.21 (A0)
- new net A1: JP3.1 (A), R2.1, U1.2 (A1)
- new net A2: JP4.1 (A), R3.1, U1.3 (A2)
- new net ex.IO0_0: U1.4 (IO0_0)
- new net ex.IO0_1: U1.5 (IO0_1)
- new net ex.IO0_2: U1.6 (IO0_2)
- new net ex.IO0_3: U1.7 (IO0_3)
- new net ex.IO0_4: U1.8 (IO0_4)
- new net ex.IO0_5: U1.9 (IO0_5)
- new net ex.IO0_6: U1.10 (IO0_6)
- new net ex.IO0_7: U1.11 (IO0_7)
- new net ex.IO1_0: U1.13 (IO1_0)
- new net ex.IO1_1: U1.14 (IO1_1)
- new net ex.IO1_2: U1.15 (IO1_2)
- new net ex.IO1_3: U1.16 (IO1_3)
- new net ex.IO1_4: U1.17 (IO1_4)
- new net ex.IO1_5: U1.18 (IO1_5)
- new net ex.IO1_6: U1.19 (IO1_6)
- new net ex.IO1_7: U1.20 (IO1_7)
- no-connect marks 5 -> 4
Other:
- added sheet Relay1 (Relay.kicad_sch)
- added sheet Relay10 (Relay.kicad_sch)
- added sheet Relay11 (Relay.kicad_sch)
- added sheet Relay12 (Relay.kicad_sch)
- added sheet Relay13 (Relay.kicad_sch)
- added sheet Relay14 (Relay.kicad_sch)
- added sheet Relay15 (Relay.kicad_sch)
- added sheet Relay16 (Relay.kicad_sch)
- added sheet Relay2 (Relay.kicad_sch)
- added sheet Relay3 (Relay.kicad_sch)
- added sheet Relay4 (Relay.kicad_sch)
- added sheet Relay5 (Relay.kicad_sch)
- added sheet Relay6 (Relay.kicad_sch)
- added sheet Relay7 (Relay.kicad_sch)
- added sheet Relay8 (Relay.kicad_sch)
- added sheet Relay9 (Relay.kicad_sch)
- title: CabHat_Template -> CabHat_relay
